Commit message: added camera, castor wheels

File: src/hitech_robot_description/urdf/hitech_robot.urdf.xacro (robot description, xacro)
@@ -127,10 +127,10 @@
     <origin xyz="0 0 0"/> <!-- Camera link mounted on the camera mount -->
   </joint>
-  <!-- Depth Camera Sensor (Stereo) -->
+  <!-- Depth Camera Sensor -->
   <gazebo reference="camera_link">
-    <sensor name="stereo_camera" type="stereo">
-      <pose>0 0 0 0 0 0</pose>
+    <sensor name="camera_link_depth_camera" type="depth">
+      <update_rate>20</update_rate>
       <camera>
-        <horizontal_fov>1.396</horizontal_fov>
+        <horizontal_fov>1.047198</horizontal_fov> <!-- 60 degrees FOV -->
         <image>
           <width>640</width>
@@ -138,17 +138,89 @@
           <format>R8G8B8</format>
         </image>
-        <depth>
-          <image>
-            <width>640</width>
-            <height>480</height>
-            <format>32FC1</format>
-          </image>
-        </depth>
         <clip>
-          <near>0.1</near>
-          <far>100.0</far>
+          <near>0.05</near>
+          <far>3</far>
         </clip>
       </camera>
+      <!-- Depth camera plugin for processing -->
+      <plugin name="camera_link_depth_controller" filename="libgazebo_ros_openni_kinect.so">
+        <baseline>0.2</baseline> <!-- Baseline for stereo camera (if used) -->
+        <alwaysOn>true</alwaysOn>
+        <updateRate>1.0</updateRate>
+        <cameraName>camera_link_ir</cameraName>
+        <imageTopicName>/camera_link/color/image_raw</imageTopicName>
+        <cameraInfoTopicName>/camera_link/color/camera_info</cameraInfoTopicName>
+        <depthImageTopicName>/camera_link/depth/image_raw</depthImageTopicName>
+        <depthImageInfoTopicName>/camera_link/depth/camera_info</depthImageInfoTopicName>
+        <pointCloudTopicName>/camera_link/depth/points</pointCloudTopicName>
+        <frameName>camera_link_frame</frameName>
+        <pointCloudCutoff>0.5</pointCloudCutoff> <!-- Minimum distance for point cloud -->
+        <pointCloudCutoffMax>3.0</pointCloudCutoffMax> <!-- Max distance for point cloud -->
+        <distortionK1>0.00000001</distortionK1>
+        <distortionK2>0.00000001</distortionK2>
+        <distortionK3>0.00000001</distortionK3>
+        <distortionT1>0.00000001</distortionT1>
+        <distortionT2>0.00000001</distortionT2>
+        <CxPrime>0</CxPrime>
+        <Cx>0</Cx>
+        <Cy>0</Cy>
+        <focalLength>0</focalLength>
+        <hackBaseline>0</hackBaseline>
+      </plugin>
     </sensor>
   </gazebo>
+  <!-- Front Caster Wheel -->
+  <link name="front_caster_wheel_link">
+    <inertial>
+      <mass value="0.1"/>
+      <inertia ixx="0.001" ixy="0.0" ixz="0.0" iyy="0.001" iyz="0.0" izz="0.001"/>
+    </inertial>
+    <visual>
+      <geometry>
+        <cylinder radius="0.03" length="0.05"/>
+      </geometry>
+      <material name="black">
+        <color rgba="0 0 0 1"/>
+      </material>
+    </visual>
+    <collision>
+      <geometry>
+        <cylinder radius="0.03" length="0.05"/>
+      </geometry>
+    </collision>
+  </link>
+  <!-- Rear Caster Wheel -->
+  <link name="rear_caster_wheel_link">
+    <inertial>
+      <mass value="0.1"/>
+      <inertia ixx="0.001" ixy="0.0" ixz="0.0" iyy="0.001" iyz="0.0" izz="0.001"/>
+    </inertial>
+    <visual>
+      <geometry>
+        <cylinder radius="0.03" length="0.05"/>
+      </geometry>
+      <material name="black">
+        <color rgba="0 0 0 1"/>
+      </material>
+    </visual>
+    <collision>
+      <geometry>
+        <cylinder radius="0.03" length="0.05"/>
+      </geometry>
+    </collision>
+  </link>
+  <!-- Joint: Base to Front Caster Wheel -->
+  <joint name="front_caster_wheel_joint" type="fixed">
+    <parent link="base_link"/>
+    <child link="front_caster_wheel_link"/>
+    <origin xyz="0.225 0 -0.075"/>
+    <axis xyz="0 1 0"/>
+  </joint>
+  <!-- Joint: Base to Rear Caster Wheel -->
+  <joint name="rear_caster_wheel_joint" type="fixed">
+    <parent link="base_link"/>
+    <child link="rear_caster_wheel_link"/>
+    <origin xyz="-0.225 0 -0.075"/>
+    <axis xyz="0 1 0"/>
+  </joint>
 </robot>

File: src/hitech_robot_description/urdf/velocity_control_gazebo.xacro (robot description, xacro)
@@ -1,5 +1,5 @@
 <?xml version="1.0"?>
 <robot name="bumperbot" xmlns:xacro="http://ros.org/wiki/xacro">
-  <!-- <transmission name="right_wheel_transmission">
+  <transmission name="right_wheel_transmission">
     <type>transmission_interface/SimpleTransmission</type>
     <joint name="right_wheel_joint" >
@@ -19,6 +19,6 @@
       <hardwareInterface>hardware_interface/VelocityJointInterface</hardwareInterface>
       <mechanicalReduction>1.0</mechanicalReduction>
-    </actuator> -->
-  <!-- </transmission> -->
+    </actuator>
+  </transmission>
   <gazebo reference="left_wheel_link">
     <mu1>1000000000000000.0</mu1>
@@ -39,10 +39,36 @@
     <fdir1>1 0 0</fdir1>
   </gazebo>
+  <gazebo reference="rear_caster_wheel_link">
+    <mu1>0.1</mu1>
+    <mu2>0.1</mu2>
+    <kp>1000000.0</kp>
+    <kd>100.0</kd>
+    <minDepth>0.001</minDepth>
+    <maxVel>1.0</maxVel>
+  </gazebo>
+  <gazebo reference="front_caster_wheel_link">
+    <mu1>0.1</mu1>
+    <mu2>0.1</mu2>
+    <kp>1000000.0</kp>
+    <kd>100.0</kd>
+    <minDepth>0.001</minDepth>
+    <maxVel>1.0</maxVel>
+  </gazebo>
   <!-- ROS Control -->
-  <!-- <gazebo>
+  <gazebo>
     <plugin name="gazebo_ros_control" filename="libgazebo_ros_control.so">
       <robotSimType>gazebo_ros_control/DefaultRobotHWSim</robotSimType>
       <legacyModeNS>true</legacyModeNS>
     </plugin>
-  </gazebo> -->
+    <!-- <plugin name="stereo_camera_plugin" filename="libgazebo_ros_camera.so">
+      <camera_name>stereo_camera</camera_name>
+      <topicName>/stereo_camera/image_raw</topicName>
+      <updateRate>30.0</updateRate>
+    </plugin> -->
+    <!-- <plugin name="mono_camera_plugin" filename="libgazebo_ros_camera.so">
+      <camera_name>mono_camera</camera_name>
+      <topicName>/mono_camera/image_raw</topicName>
+      <updateRate>30.0</updateRate>
+    </plugin> -->
+  </gazebo>
 </robot>

Commit message: added hitech robot functionality

File: src/hitech_robot_description/urdf/hitech_robot.urdf.xacro (robot description, xacro)
@@ -97,4 +97,37 @@
     </visual>
   </link>
+  <!-- Lidar Mount -->
+  <link name="lidar_mount">
+    <inertial>
+      <mass value="0.1" />
+      <inertia ixx="0.001" ixy="0.0" ixz="0.0" iyy="0.001" iyz="0.0" izz="0.001"/>
+    </inertial>
+    <visual>
+      <geometry>
+        <box size="0.1 0.1 0.025"/>
+      </geometry>
+      <origin xyz="0 0 0"/>
+      <material name="gray">
+        <color rgba="0.5 0.5 0.5 1"/> <!-- Gray Color -->
+      </material>
+    </visual>
+    <collision>
+      <geometry>
+        <box size="0.1 0.1 0.025"/>
+      </geometry>
+      <origin xyz="0 0 0"/>
+    </collision>
+  </link>
+  <!-- Lidar Link -->
+  <link name="lidar_link">
+    <visual>
+      <geometry>
+        <cylinder radius="0.05" length="0.025"/>
+      </geometry>
+      <material name="light_red">
+        <color rgba="0.5 0 0 1"/> <!-- Light red Color -->
+      </material>
+    </visual>
+  </link>
   <!-- Joint: Base to Left Wheel -->
   <joint name="left_wheel_joint" type="continuous">
@@ -126,4 +159,16 @@
     <child link="camera_link"/>
     <origin xyz="0 0 0"/> <!-- Camera link mounted on the camera mount -->
+  </joint>
+  <!-- Joint: Base to Lidar Mount (Fixed) -->
+  <joint name="lidar_mount_joint" type="fixed">
+    <parent link="base_link"/>
+    <child link="lidar_mount"/>
+    <origin xyz="-0.2 0 0.0625"/> <!-- Positioning the lidar mount above the base -->
+  </joint>
+  <!-- Camera Link to Camera Mount -->
+  <joint name="lidar_link_joint" type="fixed">
+    <parent link="lidar_mount"/>
+    <child link="lidar_link"/>
+    <origin xyz="0 0 0.0125"/> <!-- Camera link mounted on the camera mount -->
   </joint>
   <!-- Depth Camera Sensor -->
@@ -170,4 +215,36 @@
     </sensor>
   </gazebo>
+  <!-- Lidar Sensor attached to the lidar_link -->
+  <gazebo reference="lidar_link">
+    <sensor type="gpu_ray" name="lidar_sensor">
+      <pose>0 0 0 0 0 0</pose>
+      <visualize>true</visualize>
+      <update_rate>40</update_rate>
+      <ray>
+        <scan>
+          <horizontal>
+            <samples>720</samples>
+            <resolution>1</resolution>
+            <min_angle>-1.570796</min_angle>
+            <max_angle>1.570796</max_angle>
+          </horizontal>
+        </scan>
+        <range>
+          <min>0.10</min>
+          <max>30.0</max>
+          <resolution>0.01</resolution>
+        </range>
+        <noise>
+          <type>gaussian</type>
+          <mean>0.0</mean>
+          <stddev>0.01</stddev>
+        </noise>
+      </ray>
+      <plugin name="gazebo_ros_lidar_controller" filename="libgazebo_ros_gpu_laser.so">
+        <topicName>/lidar/scan</topicName>
+        <frameName>lidar_link</frameName>
+      </plugin>
+    </sensor>
+  </gazebo>
   <!-- Front Caster Wheel -->
   <link name="front_caster_wheel_link">

File: src/hitech_robot_description/urdf/velocity_control_gazebo.xacro (robot description, xacro)
@@ -61,14 +61,4 @@
       <legacyModeNS>true</legacyModeNS>
     </plugin>
-    <!-- <plugin name="stereo_camera_plugin" filename="libgazebo_ros_camera.so">
-      <camera_name>stereo_camera</camera_name>
-      <topicName>/stereo_camera/image_raw</topicName>
-      <updateRate>30.0</updateRate>
-    </plugin> -->
-    <!-- <plugin name="mono_camera_plugin" filename="libgazebo_ros_camera.so">
-      <camera_name>mono_camera</camera_name>
-      <topicName>/mono_camera/image_raw</topicName>
-      <updateRate>30.0</updateRate>
-    </plugin> -->
   </gazebo>
 </robot>

Commit message: added object in rviz

File: src/hitech_robot_description/urdf/hitech_robot.urdf.xacro (robot description, xacro)
@@ -2,5 +2,6 @@
 <robot name="hitech_robot" xmlns:xacro="http://www.ros.org/wiki/xacro">
   <xacro:include filename="$(find hitech_robot_description)/urdf/velocity_control_gazebo.xacro"/>
-  <link name="base_footprint"/>
+  <link name="base_footprint">
+  </link>
   <!-- Robot Base Link (Root Link) -->
   <link name="base_link">

File: src/hitech_robot_description/urdf/velocity_control_gazebo.xacro (robot description, xacro)
@@ -62,3 +62,16 @@
     </plugin>
   </gazebo>
+  <!-- <gazebo>
+    <plugin name="gazebo_ros_diff_drive" filename="libgazebo_ros_diff_drive.so">
+      <ros>
+        <namespace>/hitech_robot_controller</namespace>
+        <argument>cmd_vel</argument>
+      </ros>
+      <robotBaseFrame>base_footprint</robotBaseFrame>
+      <odometryFrame>odom</odometryFrame>
+      <odometryTopic>odom</odometryTopic>
+      <cmdVelTopic>/hitech_robot_controller/cmd_vel</cmdVelTopic>
+      <publishTF>true</publishTF>
+    </plugin>
+  </gazebo> -->
 </robot>
